Commit message: remove redundant estop

File: fetch_description/robots/fetch.urdf.xacro (robot description, xacro)
@@ -398,26 +398,4 @@
     <child link="bellows_link2" />
   </joint>
-  <link name="estop_link">
-    <inertial>
-      <origin rpy="0 0 0" xyz="0.002434512737072 -0.00330608315239905 0.00665139196650039" />
-      <mass value="0.00196130439134723" />
-      <inertia ixx="3.02810026604417E-07" ixy="-1.5862023118056E-08" ixz="3.16561396557437E-08" iyy="2.93322917127605E-07" iyz="-4.28833522751273E-08" izz="2.28513272627183E-07" />
-    </inertial>
-    <visual>
-      <origin rpy="0 0 0" xyz="0 0 0" />
-      <geometry>
-        <mesh filename="package://fetch_description/meshes/estop_link.STL" />
-      </geometry>
-      <material name="">
-        <color rgba="0.8 0 0 1" />
-      </material>
-    </visual>
-    <collision>
-      <origin rpy="0 0 0" xyz="0 0 0" />
-      <geometry>
-        <mesh filename="package://fetch_description/meshes/estop_link.STL" />
-      </geometry>
-    </collision>
-  </link>
   <link name="torso_fixed_link">
     <inertial>

Commit message: restore lift link

File: fetch_description/robots/fetch.urdf.xacro (robot description, xacro)
@@ -2,4 +2,26 @@
   <xacro:include filename="$(find fetch_description)/robots/macros.xacro"/>
   <xacro:freight_macro velocity_limit="17.4" />
+  <link name="torso_lift_link">
+    <inertial>
+      <origin rpy="0 0 0" xyz="-0.0013 -0.0009 0.2935" />
+      <mass value="10.7796" />
+      <inertia ixx="0.3354" ixy="0.0" ixz="-0.0162" iyx="0.0" iyy="0.3354" iyz="-0.0006" izx="-0.0162" izy="-0.0006" izz="0.0954" />
+    </inertial>
+    <visual>
+      <origin rpy="0 0 0" xyz="0 0 0" />
+      <geometry>
+        <mesh filename="package://fetch_description/meshes/torso_lift_link.dae" />
+      </geometry>
+      <material name="">
+        <color rgba="1 1 1 1" />
+      </material>
+    </visual>
+    <collision>
+      <origin rpy="0 0 0" xyz="0 0 0" />
+      <geometry>
+        <mesh filename="package://fetch_description/meshes/torso_lift_link_collision.STL" />
+      </geometry>
+    </collision>
+  </link>
   <joint name="torso_lift_joint" type="prismatic">
     <origin rpy="-6.123E-17 0 0" xyz="-0.086875 0 0.37743" />
