Commit message: new baselink mesh from rev02 gen robot added camera link and logos

File: fetch_description/robots/freight.urdf (robot description, URDF)
Before this commit: robot freight, 5 links, 4 joints
Links:
- added link base_camera_link, mass 1.52235477189066E-05; collision mesh filename=package://fetch_description/meshes/base_camera_link.DAE; visual mesh filename=package://fetch_description/meshes/base_camera_link.DAE
Joints:
- added joint base_camera_joint: type fixed, parent base_link, child base_camera_link, origin xyz=0.264511452618556 -0.00793916712988701 0.198680360086821 rpy=-6.21748940377806E-17 -0.17453292519943 1.07965570462949E-17, axis 0 0 0

Commit message: Add needed base_camera_optical_frame link/joint

File: fetch_description/robots/freight.urdf (robot description, URDF)
Before this commit: robot freight, 6 links, 5 joints
Links:
- added link base_camera_optical_frame
Joints:
- added joint base_camera_optical_joint: type fixed, parent base_camera_link, child base_camera_optical_frame, origin xyz=0 0 0 rpy=-1.5707963267966 0 0

Commit message: Fix rotation

File: fetch_description/robots/freight.urdf (robot description, URDF)
Before this commit: robot freight, 7 links, 6 joints
Joints:
- joint base_camera_joint: origin xyz=0.264511452618556 -0.00793916712988701 0.198680360086821 rpy=-6.21748940377806E-17 -0.17453292519943 1.07965570462949E-17 -> xyz=0.264511452618556 -0.00793916712988701 0.198680360086821 rpy=0 -0.17453292519943 0
- joint base_camera_optical_joint: origin xyz=0 0 0 rpy=-1.5707963267966 0 0 -> xyz=0 0 0 rpy=1.5707963267966 0 1.5707963267966

Commit message: add base camera links to freight URDF

File: fetch_description/robots/freight.urdf (robot description, URDF)
Before this commit: robot freight, 5 links, 4 joints
Links:
- added link base_camera_link
- added link base_camera_optical_frame
Joints:
- added joint base_camera_joint: type fixed, parent base_link, child base_camera_link, origin xyz=0.2645 0 0.198 rpy=0 -0.17453292519943 0
- added joint base_camera_optical_joint: type fixed, parent base_camera_link, child base_camera_optical_frame, origin xyz=0 0 0 rpy=1.5707963267966 0 1.5707963267966
