Commit message: update limits of shoulder lift joint

File: fetch_description/robots/fetch.urdf (robot description, URDF)
Before this commit: robot fetch, 26 links, 25 joints
Joints:
- joint elbow_flex_joint: limit lower=-2.26 upper=2.26 effort=66.18 velocity=1.521 -> lower=-2.251 upper=2.251 effort=66.18 velocity=1.521
- joint shoulder_lift_joint: limit lower=-3.839 upper=1.396 effort=131.76 velocity=1.454 -> lower=-1.221 upper=1.518 effort=131.76 velocity=1.454

Commit message: update velocity limits of base motors

File: fetch_description/robots/fetch.urdf (robot description, URDF)
Before this commit: robot fetch, 26 links, 25 joints
Joints:
- joint l_wheel_joint: limit effort=8.85 velocity=16.5 -> effort=8.85 velocity=17.4
- joint r_wheel_joint: limit effort=8.85 velocity=16.5 -> effort=8.85 velocity=17.4

File: fetch_description/robots/freight.urdf (robot description, URDF)
Before this commit: robot freight, 5 links, 4 joints
Joints:
- joint l_wheel_joint: limit effort=8.85 velocity=16.5 -> effort=8.85 velocity=34.8
- joint r_wheel_joint: limit effort=8.85 velocity=16.5 -> effort=8.85 velocity=34.8

Commit message: URDF says the head can tilt up 90 degrees
It is actually only ~45

File: fetch_description/robots/fetch.urdf (robot description, URDF)
Before this commit: robot fetch, 26 links, 25 joints
Joints:
- joint head_tilt_joint: limit lower=-1.57 upper=1.57 effort=0.68 velocity=1.57 -> lower=-0.785 upper=1.57 effort=0.68 velocity=1.57

Commit message: Real endstop numbers as reported by robots
min is reported in a range from -.766 to -0.863
max is reported in a range from 1.455 to 1.490

These values are conservative and should work on all existing fetch robots.

File: fetch_description/robots/fetch.urdf (robot description, URDF)
Before this commit: robot fetch, 26 links, 25 joints
Joints:
- joint head_tilt_joint: limit lower=-0.785 upper=1.57 effort=0.68 velocity=1.57 -> lower=-0.76 upper=1.45 effort=0.68 velocity=1.57

Commit message: put freight into macro, call freight macro into fetch and freight

File: fetch_description/robots/fetch.urdf (robot description, URDF)
Before this commit: robot fetch, 26 links, 25 joints
Links:
- removed link torso_lift_link

Commit message: Add generated urdf

File: fetch_description/robots/fetch.urdf (robot description, URDF)
Before this commit: robot fetch, 25 links, 25 joints
Links:
- added link torso_lift_link, mass 10.7796; collision mesh filename=package://fetch_description/meshes/torso_lift_link_collisio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; visual mesh filename=package://fetch_description/meshes/torso_lift_link.dae

Commit message: update limits of wrist flex

File: fetch_description/robots/fetch.urdf (robot description, URDF)
Before this commit: robot fetch, 26 links, 25 joints
Joints:
- joint wrist_flex_joint: limit lower=-2.18 upper=2.18 effort=25.7 velocity=2.268 -> lower=-2.16 upper=2.16 effort=25.7 velocity=2.268

Commit message: make laser actually level

File: fetch_description/robots/fetch.urdf (robot description, URDF)
Before this commit: robot fetch, 26 links, 25 joints
Joints:
- joint laser_joint: origin xyz=0.235 0 0.2878 rpy=3.1415 0 0 -> xyz=0.235 0 0.2878 rpy=3.14159265359 0 0

File: fetch_description/robots/freight.urdf (robot description, URDF)
Before this commit: robot freight, 5 links, 4 joints
Joints:
- joint laser_joint: origin xyz=0.235 0 0.2878 rpy=3.1415 0 0 -> xyz=0.235 0 0.2878 rpy=3.14159265359 0 0

Commit message: update torso throw to match rev2 hardware

File: fetch_description/robots/fetch.urdf (robot description, URDF)
Before this commit: robot fetch, 26 links, 25 joints
Joints:
- joint torso_lift_joint: limit lower=0 upper=0.4 effort=450.0 velocity=0.1 -> lower=0 upper=0.38615 effort=450.0 velocity=0.1

Commit message: added dummy link to resolve the KDL warning

File: fetch_description/robots/fetch.urdf (robot description, URDF)
Before this commit: robot fetch, 26 links, 25 joints
Links:
- added link dummy_link
Joints:
- added joint dummy_joint: type fixed, parent dummy_link, child base_link, origin xyz=0 0 0 rpy=0 0 0

Commit message: Added fixed dae models compatible with OpenGL and Minor material tweeks like red emergency button

File: fetch_description/robots/fetch.urdf (robot description, URDF)
Before this commit: robot fetch, 26 links, 25 joints
Links:
- link base_link: geometry collision mesh filename=package://fetch_description/meshes/base_link_collision.STL; visual mesh filename=package://fetch_description/meshes/base_link_fix.dae
- link elbow_flex_link: geometry collision mesh filename=package://fetch_description/meshes/elbow_flex_link_collisio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; visual mesh filename=package://fetch_description/meshes/elbow_flex_link_fix.dae
- link estop_link: geometry collision mesh filename=package://fetch_description/meshes/estop_link.STL; visual mesh filename=package://fetch_description/meshes/estop_link.dae
- link forearm_roll_link: geometry collision mesh filename=package://fetch_description/meshes/forearm_roll_link_collis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; visual mesh filename=package://fetch_description/meshes/forearm_roll_link_fix.dae
- link gripper_link: geometry collision mesh filename=package://fetch_description/meshes/gripper_link.STL; visual mesh filename=package://fetch_description/meshes/gripper_link_fix.dae
- link head_pan_link: geometry collision mesh filename=package://fetch_description/meshes/head_pan_link_collision.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; visual mesh filename=package://fetch_description/meshes/head_pan_link_fix.dae
- link head_tilt_link: geometry collision mesh filename=package://fetch_description/meshes/head_tilt_link_collision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; visual mesh filename=package://fetch_description/meshes/head_tilt_link_fix.dae
- link shoulder_lift_link: geometry collision mesh filename=package://fetch_description/meshes/shoulder_lift_link_colli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; visual mesh filename=package://fetch_description/meshes/shoulder_lift_link_fix.d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
- link shoulder_pan_link: geometry collision mesh filename=package://fetch_description/meshes/shoulder_pan_link_collis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; visual mesh filename=package://fetch_description/meshes/shoulder_pan_link_fix.dae
- link torso_fixed_link: geometry collision mesh filename=package://fetch_description/meshes/torso_fixed_link.STL; visual mesh filename=package://fetch_description/meshes/torso_fixed_link_fix.dae
- link torso_lift_link: geometry collision mesh filename=package://fetch_description/meshes/torso_lift_link_collisio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; visual mesh filename=package://fetch_description/meshes/torso_lift_link_fix.dae
- link upperarm_roll_link: geometry collision mesh filename=package://fetch_description/meshes/upperarm_roll_link_colli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; visual mesh filename=package://fetch_description/meshes/upperarm_roll_link_fix.d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
- link wrist_flex_link: geometry collision mesh filename=package://fetch_description/meshes/wrist_flex_link_collisio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; visual mesh filename=package://fetch_description/meshes/wrist_flex_link_fix.dae
- link wrist_roll_link: geometry collision mesh filename=package://fetch_description/meshes/wrist_roll_link_collisio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; visual mesh filename=package://fetch_description/meshes/wrist_roll_link_fix.dae

Commit message: Added change of names

File: fetch_description/robots/fetch.urdf (robot description, URDF)
Before this commit: robot fetch, 26 links, 25 joints
Links:
- removed link torso_fixed_link
- added link torsoed_link, mass 13.2775; collision mesh filename=package://fetch_description/meshes/torso_fixed_link.STL; visual mesh filename=package://fetch_description/meshes/torso_fixed_link.dae
- link base_link: geometry collision mesh filename=package://fetch_description/meshes/base_link_collision.STL; visual mesh filename=package://fetch_description/meshes/base_link.dae
- link elbow_flex_link: geometry collision mesh filename=package://fetch_description/meshes/elbow_flex_link_collisio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; visual mesh filename=package://fetch_description/meshes/elbow_flex_link.dae
- link forearm_roll_link: geometry collision mesh filename=package://fetch_description/meshes/forearm_roll_link_collis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; visual mesh filename=package://fetch_description/meshes/forearm_roll_link.dae
- link gripper_link: geometry collision mesh filename=package://fetch_description/meshes/gripper_link.STL; visual mesh filename=package://fetch_description/meshes/gripper_link.dae
- link head_pan_link: geometry collision mesh filename=package://fetch_description/meshes/head_pan_link_collision.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; visual mesh filename=package://fetch_description/meshes/head_pan_link.dae
- link head_tilt_link: geometry collision mesh filename=package://fetch_description/meshes/head_tilt_link_collision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; visual mesh filename=package://fetch_description/meshes/head_tilt_link.dae
- link shoulder_lift_link: geometry collision mesh filename=package://fetch_description/meshes/shoulder_lift_link_colli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; visual mesh filename=package://fetch_description/meshes/shoulder_lift_link.dae
- link shoulder_pan_link: geometry collision mesh filename=package://fetch_description/meshes/shoulder_pan_link_collis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; visual mesh filename=package://fetch_description/meshes/shoulder_pan_link.dae
- link torso_lift_link: geometry collision mesh filename=package://fetch_description/meshes/torso_lift_link_collisio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; visual mesh filename=package://fetch_description/meshes/torso_lift_link.dae
- link upperarm_roll_link: geometry collision mesh filename=package://fetch_description/meshes/upperarm_roll_link_colli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; visual mesh filename=package://fetch_description/meshes/upperarm_roll_link.dae
- link wrist_flex_link: geometry collision mesh filename=package://fetch_description/meshes/wrist_flex_link_collisio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; visual mesh filename=package://fetch_description/meshes/wrist_flex_link.dae
- link wrist_roll_link: geometry collision mesh filename=package://fetch_description/meshes/wrist_roll_link_collisio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; visual mesh filename=package://fetch_description/meshes/wrist_roll_link.dae
Joints:
- removed joint torso_fixed_joint
- added joint torsoed_joint: type fixed, parent base_link, child torsoed_link, origin xyz=-0.086875 0 0.377425 rpy=-6.12303176911189E-17 0 0, axis 0 1 0

Commit message: Fixed error in replacing names

File: fetch_description/robots/fetch.urdf (robot description, URDF)
Before this commit: robot fetch, 26 links, 25 joints
Links:
- removed link torsoed_link
- added link torso_fixed_link, mass 13.2775; collision mesh filename=package://fetch_description/meshes/torso_fixed_link.STL; visual mesh filename=package://fetch_description/meshes/torso_fixed_link.dae
Joints:
- joint torsoed_joint: child torsoed_link -> torso_fixed_link

Commit message: Update fetch.urdf

File: fetch_description/robots/fetch.urdf (robot description, URDF)
Before this commit: robot fetch, 26 links, 25 joints
Joints:
- removed joint torsoed_joint
- added joint torso_fixed_joint: type fixed, parent base_link, child torso_fixed_link, origin xyz=-0.086875 0 0.377425 rpy=-6.12303176911189E-17 0 0, axis 0 1 0
